File: kicad/power_amp.kicad_sch (KiCad schematic)
At the start: 15 parts

Commit message: Normalize BOM value strings; refresh stale top-level README
- gen_kicad NV(): normalize value strings for a tidy/consolidated BOM (2K2->2.2k,
  4K7->4.7k, drop the " film" descriptor that the footprint already conveys).
  Cosmetic only; ERC 0, demo DRC 0, SPICE exit 0, BOM regenerated.
- README rewritten to reflect the actual current state instead of the original
  reconstructed-docs snapshot: the generated + tool-verified KiCad/BOM/ngspice
  flow, the verified ~12 W power ceiling (not 18 W), the required mains fuse, the
  190x115 board + chassis-fit caveat, the active effects-chain/tone redesigns,
  and the provenance/honesty framing.

https://claude.ai/code/session_01PkrfUi9tvZfLvudJ7h23qD
Parts:
- C_in_pa: value 1uF film -> 1uF
Changed lines of the file:
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@@
     (in_bom yes) (on_board yes) (dnp no)
     (property "Reference" "C_in_pa" (at 137.16 113.02999999999999 0) (effects (font (size 1.27 1.27)) (justify left)))
-    (property "Value" "1uF film" (at 137.16 115.57 0) (effects (font (size 1.27 1.27)) (justify left)))
+    (property "Value" "1uF" (at 137.16 115.57 0) (effects (font (size 1.27 1.27)) (justify left)))
     (property "Footprint" "Capacitor_THT:C_Disc_D7.5mm_W2.5mm_P5.00mm" (at 134.62 120.64999999999999 0) (effects (font (size 1.27 1.27)) hide))
     (pin "1")
     (pin "2")
-    (instances (project "cambridge_reverb" (path "/23437dc3-547f-4e5e-a59a-04acf6aa058d" (reference "C_in_pa") (unit 1))))
+    (instances (project "cambridge_reverb" (path "/43bb109b-155d-4d3a-b8db-475f98dada40" (reference "C_in_pa") (unit 1))))
   )
   (wire (pts (xy 129.54 120.64999999999999) (xy 127.0 120.64999999999999)) (stroke (width 0) (type default)))
@@
     (pin "1")
     (pin "2")
-    (instances (project "cambridge_reverb" (path "/23437dc3-547f-4e5e-a59a-04acf6aa058d" (reference "R_bias1") (unit 1))))
+    (instances (project "cambridge_reverb" (path "/43bb109b-155d-4d3a-b8db-475f98dada40" (reference "R_bias1") (unit 1))))
   )
   (wire (pts (xy 129.54 95.25) (xy 127.0 95.25)) (stroke (width 0) (type default)))
@@
     (pin "1")
     (pin "2")
-    (instances (project "cambridge_reverb" (path "/23437dc3-547f-4e5e-a59a-04acf6aa058d" (reference "R_bias2") (unit 1))))
+    (instances (project "cambridge_reverb" (path "/43bb109b-155d-4d3a-b8db-475f98dada40" (reference "R_bias2") (unit 1))))
   )
   (wire (pts (xy 129.54 146.05) (xy 127.0 146.05)) (stroke (width 0) (type default)))
@@
     (pin "5")
     (pin "3")
-    (instances (project "cambridge_reverb" (path "/23437dc3-547f-4e5e-a59a-04acf6aa058d" (reference "IC_PA") (unit 1))))
+    (instances (project "cambridge_reverb" (path "/43bb109b-155d-4d3a-b8db-475f98dada40" (reference "IC_PA") (unit 1))))
   )
   (wire (pts (xy 193.04 128.26999999999998) (xy 190.5 128.26999999999998)) (stroke (width 0) (type default)))
@@
     (pin "1")
     (pin "2")
-    (instances (project "cambridge_reverb" (path "/23437dc3-547f-4e5e-a59a-04acf6aa058d" (reference "R_fb") (unit 1))))
+    (instances (project "cambridge_reverb" (path "/43bb109b-155d-4d3a-b8db-475f98dada40" (reference "R_fb") (unit 1))))
   )
   (wire (pts (xy 240.03 100.33) (xy 237.49 100.33)) (stroke (width 0) (type default)))
@@
     (pin "1")
     (pin "2")
-    (instances (project "cambridge_reverb" (path "/23437dc3-547f-4e5e-a59a-04acf6aa058d" (reference "C_fb_hf") (unit 1))))
+    (instances (project "cambridge_reverb" (path "/43bb109b-155d-4d3a-b8db-475f98dada40" (reference "C_fb_hf") (unit 1))))
   )
   (wire (pts (xy 240.03 81.28) (xy 237.49 81.28)) (stroke (width 0) (type default)))
@@
     (pin "1")
     (pin "2")
-    (instances (project "cambridge_reverb" (path "/23437dc3-547f-4e5e-a59a-04acf6aa058d" (reference "R_gain") (unit 1))))
+    (instances (project "cambridge_reverb" (path "/43bb109b-155d-4d3a-b8db-475f98dada40" (reference "R_gain") (unit 1))))
   )
   (wire (pts (xy 160.01999999999998 170.18) (xy 157.48 170.18)) (stroke (width 0) (type default)))
@@
     (pin "1")
     (pin "2")
-    (instances (project "cambridge_reverb" (path "/23437dc3-547f-4e5e-a59a-04acf6aa058d" (reference "C_gain") (unit 1))))
+    (instances (project "cambridge_reverb" (path "/43bb109b-155d-4d3a-b8db-475f98dada40" (reference "C_gain") (unit 1))))
   )
   (wire (pts (xy 200.66 170.18) (xy 198.12 170.18)) (stroke (width 0) (type default)))
@@
     (pin "1")
     (pin "2")
-    (instances (project "cambridge_reverb" (path "/23437dc3-547f-4e5e-a59a-04acf6aa058d" (reference "R_zobel") (unit 1))))
+    (instances (project "cambridge_reverb" (path "/43bb109b-155d-4d3a-b8db-475f98dada40" (reference "R_zobel") (unit 1))))
   )
   (wire (pts (xy 250.19 161.29) (xy 247.65 161.29)) (stroke (width 0) (type default)))
@@
     (pin "1")
     (pin "2")
-    (instances (project "cambridge_reverb" (path "/23437dc3-547f-4e5e-a59a-04acf6aa058d" (reference "C_zobel") (unit 1))))
+    (instances (project "cambridge_reverb" (path "/43bb109b-155d-4d3a-b8db-475f98dada40" (reference "C_zobel") (unit 1))))
   )
   (wire (pts (xy 280.66999999999996 161.29) (xy 278.13 161.29)) (stroke (width 0) (type default)))
@@
     (pin "1")
     (pin "2")
-    (instances (project "cambridge_reverb" (path "/23437dc3-547f-4e5e-a59a-04acf6aa058d" (reference "C_out") (unit 1))))
+    (instances (project "cambridge_reverb" (path "/43bb109b-155d-4d3a-b8db-475f98dada40" (reference "C_out") (unit 1))))
   )
   (wire (pts (xy 250.19 130.81) (xy 247.65 130.81)) (stroke (width 0) (type default)))
@@
     (pin "1")
     (pin "2")
-    (instances (project "cambridge_reverb" (path "/23437dc3-547f-4e5e-a59a-04acf6aa058d" (reference "D1") (unit 1))))
+    (instances (project "cambridge_reverb" (path "/43bb109b-155d-4d3a-b8db-475f98dada40" (reference "D1") (unit 1))))
   )
   (wire (pts (xy 240.03 200.66000000000003) (xy 237.49 200.66000000000003)) (stroke (width 0) (type default)))
@@
     (pin "1")
     (pin "2")
-    (instances (project "cambridge_reverb" (path "/23437dc3-547f-4e5e-a59a-04acf6aa058d" (reference "D2") (unit 1))))
+    (instances (project "cambridge_reverb" (path "/43bb109b-155d-4d3a-b8db-475f98dada40" (reference "D2") (unit 1))))
   )
   (wire (pts (xy 280.66999999999996 200.66000000000003) (xy 278.13 200.66000000000003)) (stroke (width 0) (type default)))
@@
     (pin "1")
     (pin "2")
-    (instances (project "cambridge_reverb" (path "/23437dc3-547f-4e5e-a59a-04acf6aa058d" (reference "C_byp1") (unit 1))))
+    (instances (project "cambridge_reverb" (path "/43bb109b-155d-4d3a-b8db-475f98dada40" (reference "C_byp1") (unit 1))))
   )
   (wire (pts (xy 129.54 200.66000000000003) (xy 127.0 200.66000000000003)) (stroke (width 0) (type default)))
@@
     (pin "1")
     (pin "2")
-    (instances (project "cambridge_reverb" (path "/23437dc3-547f-4e5e-a59a-04acf6aa058d" (reference "C_byp2") (unit 1))))
+    (instances (project "cambridge_reverb" (path "/43bb109b-155d-4d3a-b8db-475f98dada40" (reference "C_byp2") (unit 1))))
   )
   (wire (pts (xy 165.10000000000002 200.66000000000003) (xy 162.56 200.66000000000003)) (stroke (width 0) (type default)))
