File: kicad/power_section_demo.kicad_pcb (KiCad board)
At the start: 2 copper layers, 120 x 70 mm, 8 parts, among them U1 LM317T

Commit message: Keep LM317-input pre-filter (rename +27V->VREG_IN, 47R->100R) - corrected call
On reflection my earlier "delete R_27V, feed LM317 from +33.5V" recommendation
was wrong for a noise-conscious design: R_27V + C_filt1 is an RC pre-filter on
the LM317 input AND decouples the preamp supply from the power amp's transient
current draw on the +33.5V rail (the LM317's PSRR alone falls off with
frequency). Deleting it would hurt noise.

The real bug was the mislabeling: under the modern ~15 mA load the node sits at
~32 V, not 27 V, so the "27 V rail / 26-28 V" naming was a leftover misnomer.

Done instead:
- keep the element; bump 47R/2W -> 100R/1W (~6 dB more 120 Hz ripple rejection,
  ~1.5 V drop at 15 mA, LM317 in-out diff 14.7 V << 40 V max, ~0.02 W)
- rename net +27V -> VREG_IN (schematic gen, .kicad_pro Power pattern)
- correct the docs/troubleshooting voltages (~31-33 V) across Part 1/2/3/4,
  errata, BOM, availability-audit, PCB-NOTES/AUDIT, SCHEMATIC-BUILD, CHECKLIST

Verified: sch erc 0, full DRC unchanged (164), demo DRC 0, SPICE exit 0, BOM
CSV clean, net classes intact (VREG_IN now in the Power pattern).

https://claude.ai/code/session_01PkrfUi9tvZfLvudJ7h23qD
Parts:
- R_27V: value 47R/2W -> 100R/1W
Connections:
- net +27V renamed VREG_IN

Commit message: Redesign effects chain: active reverb summer + output buffer + split bias
Resolves roast R3 (broken passive mixer) and R6 (shared VBIAS bleed), using the
two spare TL072 halves and verifying with a rail-aware SPICE model.

- Reverb wet/dry mix is now an ACTIVE inverting summer on IC1-B (dry always on,
  wet via POT_REV, unity each, low-Z out about VBIAS_R). Removed the broken
  passive R_dry_tap/R_blend1/R_blend2 (1M dry series made it ~all-wet into an
  unbuffered 110k node).
- IC2-B repurposed as the post-MRB OUTPUT BUFFER driving PA_IN (removed the
  unbuffered R_painput 1M and a dead C_trem_out/R_trem_pass branch).
- VBIAS split into independent VBIAS_R (reverb) and VBIAS_T (tremolo) dividers
  (100k/100k + 47uF each) -> the LFO can no longer modulate the reverb reference.

Verification: new models/opamp_rail.sub clamps the output to the rails (unlike
opamp1p.sub), and spice/tran_reverb_mixer.cir confirms on a single +17V supply:
mid-rail bias 8.50 V, unity (0.0 dB) sum, clips at 15.5/1.5 V -> +-7 V headroom
(~24 dB over a 0.42 V program peak). This is the large-signal/headroom check the
rail-less model could not do (roast R7).

ERC 0; demo DRC 0; full board regenerated (106 footprints); run_all.sh exit 0;
BOM + roast doc + SCHEMATIC-BUILD + spice/README + CHANGELOG updated.

https://claude.ai/code/session_01PkrfUi9tvZfLvudJ7h23qD
Parts:
- removed R_vb1: 100k, R_Axial_DIN0207_L6.3mm_D2.5mm_P5.08mm_Vertical
- added R_vbr1: 100k, R_Axial_DIN0207_L6.3mm_D2.5mm_P5.08mm_Vertical, F.Cu at (94.0, 48.0)
