File: kicad/tremolo.kicad_sch (KiCad schematic)
At the start: 18 parts, among them IC2 TL072CP

Commit message: Generate BOM from schematic (authoritative); complete missing schematic parts
The BOM had drifted badly from the schematic (~20 parts in the schematic missing
from the BOM, ~20 stale/renamed rows in the BOM). Root-caused two ways:

1. Completed the SCHEMATIC -- added parts that were in Part 2 / the BOM but never
   actually placed: rectifier snubbers C101-C104, 2nd pre-filter C_filt2, and the
   tremolo SPEED/DEPTH pots (POT_SPD as a rheostat in the Wien series arm to vary
   frequency; POT_DPT scaling the LFO into the VTL1 LED for depth). 117 comps, ERC 0.

2. Made the BOM GENERATED from the schematic: kicad/gen/gen_bom.py emits bom/bom.csv
   per-reference 1:1 with the netlist (verified: every schematic ref present),
   merged with curated part numbers/notes and an explicit off-board/mechanical
   section (sockets, heatsink, mica, standoffs, fuses, mains fuse). Also writes
   bom/bom-grouped.csv (consolidated by value+footprint for ordering). bom/README
   updated to say it's generated; do not hand-edit.

Verified: sch erc 0, demo DRC 0, run_all.sh exit 0, BOM 8-col clean, every
schematic ref covered. Full board now 113 footprints; density 53%/90% (190x115 /
155x90) -- reinforces the chassis-fit finding.

https://claude.ai/code/session_01PkrfUi9tvZfLvudJ7h23qD
Parts:
- added POT_DPT: 100k lin, Connector_PinHeader_2.54mm:PinHeader_1x03_P2.54mm_Vertical, symbol cr_primitives:POT
- added POT_SPD: 500k lin, Connector_PinHeader_2.54mm:PinHeader_1x03_P2.54mm_Vertical, symbol cr_primitives:POT
- R_lfo_ser: value 100k -> 10k
Connections:
- net LFO_OUT: now also POT_DPT.1; no longer R_led.1
- net VBIAS_T: now also POT_DPT.3
- net WN1: now also POT_SPD.2 (W), POT_SPD.3; no longer R_lfo_ser.2
- new net DPT_W: POT_DPT.2 (W), R_led.1
- new net SPD_A: POT_SPD.1, R_lfo_ser.2

Commit message: Normalize BOM value strings; refresh stale top-level README
- gen_kicad NV(): normalize value strings for a tidy/consolidated BOM (2K2->2.2k,
  4K7->4.7k, drop the " film" descriptor that the footprint already conveys).
  Cosmetic only; ERC 0, demo DRC 0, SPICE exit 0, BOM regenerated.
- README rewritten to reflect the actual current state instead of the original
  reconstructed-docs snapshot: the generated + tool-verified KiCad/BOM/ngspice
  flow, the verified ~12 W power ceiling (not 18 W), the required mains fuse, the
  190x115 board + chassis-fit caveat, the active effects-chain/tone redesigns,
  and the provenance/honesty framing.

https://claude.ai/code/session_01PkrfUi9tvZfLvudJ7h23qD
Parts:
- R_led_diag: value 2K2 -> 2.2k
- R_lfo_fb2: value 4K7 -> 4.7k
Changed lines of the file:
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@@
     (pin "8")
     (pin "4")
-    (instances (project "cambridge_reverb" (path "/2dfdb826-abc1-4406-b599-c9ec64880de4" (reference "IC2") (unit 1))))
+    (instances (project "cambridge_reverb" (path "/d42230cc-952b-4e7b-8b81-b7cfcd0de5be" (reference "IC2") (unit 1))))
   )
   (wire (pts (xy 191.76999999999998 116.84) (xy 189.23 116.84)) (stroke (width 0) (type default)))
@@
     (pin "1")
     (pin "2")
-    (instances (project "cambridge_reverb" (path "/2dfdb826-abc1-4406-b599-c9ec64880de4" (reference "C_obuf_in") (unit 1))))
+    (instances (project "cambridge_reverb" (path "/d42230cc-952b-4e7b-8b81-b7cfcd0de5be" (reference "C_obuf_in") (unit 1))))
   )
   (wire (pts (xy 119.38 71.12) (xy 116.84 71.12)) (stroke (width 0) (type default)))
@@
     (pin "1")
     (pin "2")
-    (instances (project "cambridge_reverb" (path "/2dfdb826-abc1-4406-b599-c9ec64880de4" (reference "R_obuf_b") (unit 1))))
+    (instances (project "cambridge_reverb" (path "/d42230cc-952b-4e7b-8b81-b7cfcd0de5be" (reference "R_obuf_b") (unit 1))))
   )
   (wire (pts (xy 119.38 101.6) (xy 116.84 101.6)) (stroke (width 0) (type default)))
@@
     (pin "1")
     (pin "2")
-    (instances (project "cambridge_reverb" (path "/2dfdb826-abc1-4406-b599-c9ec64880de4" (reference "R_lfo_ser") (unit 1))))
+    (instances (project "cambridge_reverb" (path "/d42230cc-952b-4e7b-8b81-b7cfcd0de5be" (reference "R_lfo_ser") (unit 1))))
   )
   (wire (pts (xy 228.59999999999997 86.36) (xy 226.06 86.36)) (stroke (width 0) (type default)))
@@
     (pin "3")
     (pin "2")
-    (instances (project "cambridge_reverb" (path "/2dfdb826-abc1-4406-b599-c9ec64880de4" (reference "POT_SPD") (unit 1))))
+    (instances (project "cambridge_reverb" (path "/d42230cc-952b-4e7b-8b81-b7cfcd0de5be" (reference "POT_SPD") (unit 1))))
   )
   (wire (pts (xy 259.08 86.36) (xy 256.54 86.36)) (stroke (width 0) (type default)))
@@
     (pin "1")
     (pin "2")
-    (instances (project "cambridge_reverb" (path "/2dfdb826-abc1-4406-b599-c9ec64880de4" (reference "C_lfo1") (unit 1))))
+    (instances (project "cambridge_reverb" (path "/d42230cc-952b-4e7b-8b81-b7cfcd0de5be" (reference "C_lfo1") (unit 1))))
   )
   (wire (pts (xy 288.28999999999996 91.44) (xy 285.75 91.44)) (stroke (width 0) (type default)))
@@
     (pin "1")
     (pin "2")
-    (instances (project "cambridge_reverb" (path "/2dfdb826-abc1-4406-b599-c9ec64880de4" (reference "R_lfo1") (unit 1))))
+    (instances (project "cambridge_reverb" (path "/d42230cc-952b-4e7b-8b81-b7cfcd0de5be" (reference "R_lfo1") (unit 1))))
   )
   (wire (pts (xy 238.76 151.13) (xy 236.22000000000003 151.13)) (stroke (width 0) (type default)))
@@
     (pin "1")
     (pin "2")
-    (instances (project "cambridge_reverb" (path "/2dfdb826-abc1-4406-b599-c9ec64880de4" (reference "C_lfo2") (unit 1))))
+    (instances (project "cambridge_reverb" (path "/d42230cc-952b-4e7b-8b81-b7cfcd0de5be" (reference "C_lfo2") (unit 1))))
   )
   (wire (pts (xy 274.32 151.13) (xy 271.78 151.13)) (stroke (width 0) (type default)))
@@
     (pin "1")
     (pin "2")
-    (instances (project "cambridge_reverb" (path "/2dfdb826-abc1-4406-b599-c9ec64880de4" (reference "R_lfo_fb1") (unit 1))))
+    (instances (project "cambridge_reverb" (path "/d42230cc-952b-4e7b-8b81-b7cfcd0de5be" (reference "R_lfo_fb1") (unit 1))))
   )
   (wire (pts (xy 158.75 101.6) (xy 156.21 101.6)) (stroke (width 0) (type default)))
@@
     (in_bom yes) (on_board yes) (dnp no)
     (property "Reference" "R_lfo_fb2" (at 166.36999999999998 134.62 0) (effects (font (size 1.27 1.27)) (justify left)))
-    (property "Value" "4K7" (at 166.36999999999998 137.16 0) (effects (font (size 1.27 1.27)) (justify left)))
+    (property "Value" "4.7k" (at 166.36999999999998 137.16 0) (effects (font (size 1.27 1.27)) (justify left)))
     (property "Footprint" "Resistor_THT:R_Axial_DIN0207_L6.3mm_D2.5mm_P5.08mm_Vertical" (at 163.82999999999998 142.24 0) (effects (font (size 1.27 1.27)) hide))
     (pin "1")
     (pin "2")
-    (instances (project "cambridge_reverb" (path "/2dfdb826-abc1-4406-b599-c9ec64880de4" (reference "R_lfo_fb2") (unit 1))))
+    (instances (project "cambridge_reverb" (path "/d42230cc-952b-4e7b-8b81-b7cfcd0de5be" (reference "R_lfo_fb2") (unit 1))))
   )
   (wire (pts (xy 158.75 142.24) (xy 156.21 142.24)) (stroke (width 0) (type default)))
@@
     (pin "1")
     (pin "2")
-    (instances (project "cambridge_reverb" (path "/2dfdb826-abc1-4406-b599-c9ec64880de4" (reference "D_lfo1") (unit 1))))
+    (instances (project "cambridge_reverb" (path "/d42230cc-952b-4e7b-8b81-b7cfcd0de5be" (reference "D_lfo1") (unit 1))))
   )
   (wire (pts (xy 128.27 101.6) (xy 125.73 101.6)) (stroke (width 0) (type default)))
@@
     (pin "1")
     (pin "2")
-    (instances (project "cambridge_reverb" (path "/2dfdb826-abc1-4406-b599-c9ec64880de4" (reference "D_lfo2") (unit 1))))
+    (instances (project "cambridge_reverb" (path "/d42230cc-952b-4e7b-8b81-b7cfcd0de5be" (reference "D_lfo2") (unit 1))))
   )
   (wire (pts (xy 128.27 132.07999999999998) (xy 125.73 132.07999999999998)) (stroke (width 0) (type default)))
@@
     (pin "3")
     (pin "2")
-    (instances (project "cambridge_reverb" (path "/2dfdb826-abc1-4406-b599-c9ec64880de4" (reference "POT_DPT") (unit 1))))
+    (instances (project "cambridge_reverb" (path "/d42230cc-952b-4e7b-8b81-b7cfcd0de5be" (reference "POT_DPT") (unit 1))))
   )
   (wire (pts (xy 204.47 181.61) (xy 201.93 181.61)) (stroke (width 0) (type default)))
@@
     (pin "1")
     (pin "2")
-    (instances (project "cambridge_reverb" (path "/2dfdb826-abc1-4406-b599-c9ec64880de4" (reference "R_led") (unit 1))))
+    (instances (project "cambridge_reverb" (path "/d42230cc-952b-4e7b-8b81-b7cfcd0de5be" (reference "R_led") (unit 1))))
   )
   (wire (pts (xy 243.83999999999997 181.61) (xy 241.3 181.61)) (stroke (width 0) (type default)))
@@
     (pin "3")
     (pin "4")
-    (instances (project "cambridge_reverb" (path "/2dfdb826-abc1-4406-b599-c9ec64880de4" (reference "VTL1") (unit 1))))
+    (instances (project "cambridge_reverb" (path "/d42230cc-952b-4e7b-8b81-b7cfcd0de5be" (reference "VTL1") (unit 1))))
   )
   (wire (pts (xy 285.75 179.07000000000002) (xy 283.21 179.07000000000002)) (stroke (width 0) (type default)))
@@
     (in_bom yes) (on_board yes) (dnp no)
     (property "Reference" "R_led_diag" (at 246.38000000000002 204.47 0) (effects (font (size 1.27 1.27)) (justify left)))
-    (property "Value" "2K2" (at 246.38000000000002 207.01 0) (effects (font (size 1.27 1.27)) (justify left)))
+    (property "Value" "2.2k" (at 246.38000000000002 207.01 0) (effects (font (size 1.27 1.27)) (justify left)))
     (property "Footprint" "Resistor_THT:R_Axial_DIN0207_L6.3mm_D2.5mm_P5.08mm_Vertical" (at 243.84000000000003 212.09 0) (effects (font (size 1.27 1.27)) hide))
     (pin "1")
     (pin "2")
-    (instances (project "cambridge_reverb" (path "/2dfdb826-abc1-4406-b599-c9ec64880de4" (reference "R_led_diag") (unit 1))))
+    (instances (project "cambridge_reverb" (path "/d42230cc-952b-4e7b-8b81-b7cfcd0de5be" (reference "R_led_diag") (unit 1))))
   )
   (wire (pts (xy 238.76 212.09) (xy 236.22000000000003 212.09)) (stroke (width 0) (type default)))
@@
     (pin "1")
     (pin "2")
-    (instances (project "cambridge_reverb" (path "/2dfdb826-abc1-4406-b599-c9ec64880de4" (reference "LED_rate") (unit 1))))
+    (instances (project "cambridge_reverb" (path "/d42230cc-952b-4e7b-8b81-b7cfcd0de5be" (reference "LED_rate") (unit 1))))
   )
   (wire (pts (xy 284.48 212.09) (xy 281.94 212.09)) (stroke (width 0) (type default)))
@@
     (pin "1")
     (pin "2")
-    (instances (project "cambridge_reverb" (path "/2dfdb826-abc1-4406-b599-c9ec64880de4" (reference "R_trem1") (unit 1))))
+    (instances (project "cambridge_reverb" (path "/d42230cc-952b-4e7b-8b81-b7cfcd0de5be" (reference "R_trem1") (unit 1))))
   )
   (wire (pts (xy 148.59 181.61) (xy 146.05 181.61)) (stroke (width 0) (type default)))
@@
     (pin "1")
     (pin "2")
-    (instances (project "cambridge_reverb" (path "/2dfdb826-abc1-4406-b599-c9ec64880de4" (reference "C_dc_blk") (unit 1))))
+    (instances (project "cambridge_reverb" (path "/d42230cc-952b-4e7b-8b81-b7cfcd0de5be" (reference "C_dc_blk") (unit 1))))
   )
   (wire (pts (xy 148.59 212.09) (xy 146.05 212.09)) (stroke (width 0) (type default)))
@@
     (pin "1")
     (pin "2")
-    (instances (project "cambridge_reverb" (path "/2dfdb826-abc1-4406-b599-c9ec64880de4" (reference "R_fs_trem") (unit 1))))
+    (instances (project "cambridge_reverb" (path "/d42230cc-952b-4e7b-8b81-b7cfcd0de5be" (reference "R_fs_trem") (unit 1))))
   )
   (wire (pts (xy 119.38 212.09) (xy 116.84 212.09)) (stroke (width 0) (type default)))
