File: kicad/tremolo.kicad_sch (KiCad schematic)
At the start: 26 parts, among them IC2 TL072CP

Commit message: Noise, hum, crosstalk and thermal models; three design fixes; JLCPCB rules and cost
New models (docs/06c, spice/): a .noise run of the whole front end including the
LM317's own rail noise, the rail-ripple paths to the speaker, a vactrol-level tremolo
depth model, an electro-thermal LM1875 ladder, and a geometric crosstalk audit of the
routed boards (kicad/gen/crosstalk_audit.py). They found three defects:

- Errata #21 (hum + hiss): the LM1875 bias divider had no bypass (+4 dB ripple to
  speaker, 0.4 Vrms of 100 Hz at idle) and the LM317's 0.5 mV of noise reached the
  0 dB-PSRR JFET stages (23 dB above their floor, SNR 34 dB). Fixed with C_bref +
  R_bias3 on the power amp, C_adj on the regulator, and an RC-decoupled +17V_PRE rail
  for Q1/Q2/Q_rec: hum 408 mV -> 0.3 mV, EIN 37 -> 2.7 uV, SNR 34 -> 57 dB.
- Errata #22 (tremolo depth 1.7 dB): the vactrol LED was returned to ground from a
  mid-rail LFO -> 7 mA DC, a fixed -20 dB pad. LED limiter (2 V swing, LED_rate is one
  limiter LED) + Q_trem 2N3904/MMBT3904 emitter follower AC-coupled from the depth
  pot -> 15 dB depth, 0.8 dB insertion loss.
- Errata #23 (fab): stock TO-92 and the LM1875 footprint were under JLCPCB's 0.18 mm
  annular-ring minimum -> TO-92_Inline_Wide and 1.5 mm LM1875 pads; both .kicad_pro
  carry JLC's 2-layer limits as DRC constraints. Cost: all SMD caps 1206 (basic
  library), "(opt)" MRB caps DNP, gyrator on E24 values (same 1.86 H): 7 -> 2
  extended part types, ~$32 -> ~$17 assembly for five boards (kicad/gen/jlc_cost.py);
  three fiducials on the SMD board.

Crosstalk -> two routing rules (.kicad_dru: HighCurrent 0.6/0.4 mm and TankDrive
1.2/0.8 mm from signal copper, THT/SMD) that route_board.py also hands the router as
class clearances; keepout rule areas along the edge and around the mounting holes.
Thermal: Part 5's <= 2.5 K/W heatsink confirmed with numbers (Tj 97 C at 40 C ambient,
worst-case sine; 8-10 K/W clip-ons reach shutdown).

Placer: short parts stack beside tall ones i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
Parts:
- removed D_lfo1, D_lfo2: 1N4148, Diode_THT:D_DO-41_SOD81_P10.16mm_Horizontal, symbol cr_primitives:D
- removed R_led: 1k, Resistor_THT:R_Axial_DIN0207_L6.3mm_D2.5mm_P5.08mm_Vertical, symbol cr_primitives:R
- removed R_led_diag: 2.2k, Resistor_THT:R_Axial_DIN0207_L6.3mm_D2.5mm_P5.08mm_Vertical, symbol cr_primitives:R
- added C_drv: 100uF/25V, Capacitor_THT:CP_Radial_D6.3mm_P2.50mm, symbol cr_primitives:CP
- added LED_lim: 3mm red, LED_THT:LED_D3.0mm, symbol cr_primitives:LED
- added Q_trem: 2N3904, Package_TO_SOT_THT:TO-92_Inline_Wide, symbol cr_primitives:NPN
- added R_b1: 180k, Resistor_THT:R_Axial_DIN0207_L6.3mm_D2.5mm_P5.08mm_Vertical, symbol cr_primitives:R
- added R_b2: 10k, Resistor_THT:R_Axial_DIN0207_L6.3mm_D2.5mm_P5.08mm_Vertical, symbol cr_primitives:R
- added R_c: 100R, Resistor_THT:R_Axial_DIN0207_L6.3mm_D2.5mm_P5.08mm_Vertical, symbol cr_primitives:R
- added R_e: 470R, Resistor_THT:R_Axial_DIN0207_L6.3mm_D2.5mm_P5.08mm_Vertical, symbol cr_primitives:R
Connections:
- net DLED is gone; now on net LFO_OUT: LED_rate.1 (A)
- net +17V: now also R_b1.1, R_c.1
- net DPT_W: now also C_drv.1 (+)
- net GND: now also R_b2.2, R_e.2; no longer LED_rate.2 (K), VTL1.2 (LED_K)
- net LFO_N: now also LED_rate.2 (K), LED_lim.1 (A)
- net LFO_OUT: now also LED_lim.2 (K)
- net VLED: now also R_c.2
- new net QB: C_drv.2, Q_trem.2 (B), R_b1.2, R_b2.1
- new net QC: Q_trem.3 (C), VTL1.2 (LED_K)
- new net QE: Q_trem.1 (E), R_e.1
Other:
- note added: "TREMOLO -- IC2-A: Wien LFO (0.6-10.6 Hz), limited by two antiparallel LEDs (~2 V swing; LED_rate blinks). Q_trem: AC-coupled emitter follower drives the VTL5C1 LED 0..6 mA -> 15 dB depth, 0.8 dB insertion loss (was 7 mA DC: -20 dB pad, 1.7 dB depth). IC2-B: post-MRB output buffer -> PA_IN."
- note removed: "TREMOLO -- IC2-A: Wien LFO (~16Hz) -> VTL5C1. IC2-B: post-MRB output buffer -> PA_IN. All on VBIAS_T."
