File: kicad/power_amp_classa.kicad_sch (KiCad schematic)
At the start: 20 parts

Commit message: Datasheet footprints, floor-plan placement, headless autoroute (144/145, DRC 0)
PCB-AUDIT s1 fixes with datasheet-derived project footprints:
- TO-220-5_Vertical_P1.70mm_LM1875 (TI NDH0005D): 1.45 mm pads on the 1.1 mm
  drill -> 0.175 mm annular (was 0.0875, 5 DRC errors); pad-local 0.2 mm clearance
- Bridge_KBP_P3.81mm (Diodes DS39310 KBP404G-KBP410G, pins + ~ ~ -); bridge
  symbol renumbered to the physical order; errata #3 updated (KBU needs a swap)
- value-aware CP/R sizing (real can sizes for 4700/2200/1000 uF, 5 W / 1 W
  resistors, fat pads on the 0R speaker return); Part 4 wire pads for all
  off-board wiring (2.0 mm/1.2 mm signal, 3.0 mm/1.5 mm speaker + transformer)
- VRAW/AC1/AC2 moved into the HighCurrent net class (errata #11)

gen_pcb.py now places to the Part 5 floor plan: balanced columns (Input/Preamp
with Tone stacked below | Reverb/Trem/MRB | Power Amp | PSU), signal order inside
zones with serpentine shelves, LM1875/LM317 on the top edge with the 10 mm
keep-out, wiring edge along the bottom, 4x M3 holes, two locked 0.9 mm escape
stubs off the LM1875 pins 4/5 (a 1.5/2.5 mm trace cannot enter a 1.70 mm pitch).
DRC before routing: 0 errors, 0 warnings.

route_board.py: pcbnew DSN export -> Freerouting -> SES import -> pour refill.
Freerouting 2.1.0 ignores every pass/timeout limit in CLI mode and only writes
output at 0 unrouted (and its MT router crashed), so the script drives 1.9.0
under xvfb-run and injects autoroute_settings (bottom layer 6x cost, via 80) so
the GND pour stays whole. Committed board: 144/145 connections routed, 0 DRC
violations (--severity-all), 26 vias, 351 mm on the bottom vs 3.7 m on top; the
one open PA_OUT link (blocked by R_bias1) is documented as a GUI finish.

Chassis-fit figure corrected: the old 48-53 % / 82-90 % densities counted hidden
text boxes; text-less it is ~33 % on 190x115 and ~56 % on 155x90.

Docs: PCB-NOTES/PCB-AUDIT rewritten, README, CHANGELOG, errata #3/#11,
SOURCES (package drawings), Part 10, kicad RE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
Parts:
- C_byp2, C_gain: footprint Capacitor_THT:CP_Radial_D8.0mm_P3.50mm -> Capacitor_THT:CP_Radial_D5.0mm_P2.00mm
- C_out: footprint Capacitor_THT:CP_Radial_D8.0mm_P3.50mm -> Capacitor_THT:CP_Radial_D16.0mm_P7.50mm
- IC_PA: footprint Package_TO_SOT_THT:TO-220-5_Vertical -> cambridge_reverb:TO-220-5_Vertical_P1.70mm_LM1875
- R_spk_rtn: footprint Resistor_THT:R_Axial_DIN0207_L6.3mm_D2.5mm_P5.08mm_Vertical -> Resistor_THT:R_Axial_DIN0414_L11.9mm_D4.5mm_P15.24mm_Horizontal
