File: kicad/switching.kicad_sch (KiCad schematic)
At the start: 6 parts

Commit message: Datasheet footprints, floor-plan placement, headless autoroute (144/145, DRC 0)
PCB-AUDIT s1 fixes with datasheet-derived project footprints:
- TO-220-5_Vertical_P1.70mm_LM1875 (TI NDH0005D): 1.45 mm pads on the 1.1 mm
  drill -> 0.175 mm annular (was 0.0875, 5 DRC errors); pad-local 0.2 mm clearance
- Bridge_KBP_P3.81mm (Diodes DS39310 KBP404G-KBP410G, pins + ~ ~ -); bridge
  symbol renumbered to the physical order; errata #3 updated (KBU needs a swap)
- value-aware CP/R sizing (real can sizes for 4700/2200/1000 uF, 5 W / 1 W
  resistors, fat pads on the 0R speaker return); Part 4 wire pads for all
  off-board wiring (2.0 mm/1.2 mm signal, 3.0 mm/1.5 mm speaker + transformer)
- VRAW/AC1/AC2 moved into the HighCurrent net class (errata #11)

gen_pcb.py now places to the Part 5 floor plan: balanced columns (Input/Preamp
with Tone stacked below | Reverb/Trem/MRB | Power Amp | PSU), signal order inside
zones with serpentine shelves, LM1875/LM317 on the top edge with the 10 mm
keep-out, wiring edge along the bottom, 4x M3 holes, two locked 0.9 mm escape
stubs off the LM1875 pins 4/5 (a 1.5/2.5 mm trace cannot enter a 1.70 mm pitch).
DRC before routing: 0 errors, 0 warnings.

route_board.py: pcbnew DSN export -> Freerouting -> SES import -> pour refill.
Freerouting 2.1.0 ignores every pass/timeout limit in CLI mode and only writes
output at 0 unrouted (and its MT router crashed), so the script drives 1.9.0
under xvfb-run and injects autoroute_settings (bottom layer 6x cost, via 80) so
the GND pour stays whole. Committed board: 144/145 connections routed, 0 DRC
violations (--severity-all), 26 vias, 351 mm on the bottom vs 3.7 m on top; the
one open PA_OUT link (blocked by R_bias1) is documented as a GUI finish.

Chassis-fit figure corrected: the old 48-53 % / 82-90 % densities counted hidden
text boxes; text-less it is ~33 % on 190x115 and ~56 % on 155x90.

Docs: PCB-NOTES/PCB-AUDIT rewritten, README, CHANGELOG, errata #3/#11,
SOURCES (package drawings), Part 10, kicad RE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
Parts:
- FS1: footprint Connector_PinHeader_2.54mm:PinHeader_1x06_P2.54mm_Vertical -> cambridge_reverb:WirePad_1x06_P2.54mm_D1.2mm
- J_IN1, J_IN2, J_IN3: footprint Connector_PinHeader_2.54mm:PinHeader_1x02_P2.54mm_Vertical -> cambridge_reverb:WirePad_1x02_P2.54mm_D1.2mm
- LS1: footprint Connector_PinHeader_2.54mm:PinHeader_1x02_P2.54mm_Vertical -> cambridge_reverb:WirePad_1x02_P5.08mm_D1.5mm
- R_spk_rtn: footprint Resistor_THT:R_Axial_DIN0207_L6.3mm_D2.5mm_P5.08mm_Vertical -> Resistor_THT:R_Axial_DIN0414_L11.9mm_D4.5mm_P15.24mm_Horizontal
Changed lines of the file:
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@@
     (property "Reference" "J_IN1" (at 137.16 88.89999999999999 0) (effects (font (size 1.27 1.27)) (justify left)))
     (property "Value" "Input 1" (at 137.16 91.44 0) (effects (font (size 1.27 1.27)) (justify left)))
-    (property "Footprint" "Connector_PinHeader_2.54mm:PinHeader_1x02_P2.54mm_Vertical" (at 134.62 96.52 0) (effects (font (size 1.27 1.27)) hide))
+    (property "Footprint" "cambridge_reverb:WirePad_1x02_P2.54mm_D1.2mm" (at 134.62 96.52 0) (effects (font (size 1.27 1.27)) hide))
     (pin "1")
     (pin "2")
-    (instances (project "cambridge_reverb" (path "/bb8f46f8-d0af-4906-93ac-5291092b4687" (reference "J_IN1") (unit 1))))
+    (instances (project "cambridge_reverb" (path "/3395a9cf-4e5b-48c0-af92-0653b32bf036" (reference "J_IN1") (unit 1))))
   )
   (wire (pts (xy 139.7 93.97999999999999) (xy 142.24 93.97999999999999)) (stroke (width 0) (type default)))
@@
     (property "Reference" "J_IN2" (at 137.16 119.38 0) (effects (font (size 1.27 1.27)) (justify left)))
     (property "Value" "Input 2" (at 137.16 121.92 0) (effects (font (size 1.27 1.27)) (justify left)))
-    (property "Footprint" "Connector_PinHeader_2.54mm:PinHeader_1x02_P2.54mm_Vertical" (at 134.62 127.0 0) (effects (font (size 1.27 1.27)) hide))
+    (property "Footprint" "cambridge_reverb:WirePad_1x02_P2.54mm_D1.2mm" (at 134.62 127.0 0) (effects (font (size 1.27 1.27)) hide))
     (pin "1")
     (pin "2")
-    (instances (project "cambridge_reverb" (path "/bb8f46f8-d0af-4906-93ac-5291092b4687" (reference "J_IN2") (unit 1))))
+    (instances (project "cambridge_reverb" (path "/3395a9cf-4e5b-48c0-af92-0653b32bf036" (reference "J_IN2") (unit 1))))
   )
   (wire (pts (xy 139.7 124.46) (xy 142.24 124.46)) (stroke (width 0) (type default)))
@@
     (property "Reference" "J_IN3" (at 137.16 148.58999999999997 0) (effects (font (size 1.27 1.27)) (justify left)))
     (property "Value" "IN3 / FX return" (at 137.16 151.12999999999997 0) (effects (font (size 1.27 1.27)) (justify left)))
-    (property "Footprint" "Connector_PinHeader_2.54mm:PinHeader_1x02_P2.54mm_Vertical" (at 134.62 156.20999999999998 0) (effects (font (size 1.27 1.27)) hide))
+    (property "Footprint" "cambridge_reverb:WirePad_1x02_P2.54mm_D1.2mm" (at 134.62 156.20999999999998 0) (effects (font (size 1.27 1.27)) hide))
     (pin "1")
     (pin "2")
-    (instances (project "cambridge_reverb" (path "/bb8f46f8-d0af-4906-93ac-5291092b4687" (reference "J_IN3") (unit 1))))
+    (instances (project "cambridge_reverb" (path "/3395a9cf-4e5b-48c0-af92-0653b32bf036" (reference "J_IN3") (unit 1))))
   )
   (wire (pts (xy 139.7 153.67) (xy 142.24 153.67)) (stroke (width 0) (type default)))
@@
     (property "Reference" "FS1" (at 227.33 119.38 0) (effects (font (size 1.27 1.27)) (justify left)))
     (property "Value" "DIN-6" (at 227.33 121.92 0) (effects (font (size 1.27 1.27)) (justify left)))
-    (property "Footprint" "Connector_PinHeader_2.54mm:PinHeader_1x06_P2.54mm_Vertical" (at 224.79000000000002 127.0 0) (effects (font (size 1.27 1.27)) hide))
+    (property "Footprint" "cambridge_reverb:WirePad_1x06_P2.54mm_D1.2mm" (at 224.79000000000002 127.0 0) (effects (font (size 1.27 1.27)) hide))
     (pin "1")
     (pin "2")
@@
     (pin "5")
     (pin "6")
-    (instances (project "cambridge_reverb" (path "/bb8f46f8-d0af-4906-93ac-5291092b4687" (reference "FS1") (unit 1))))
+    (instances (project "cambridge_reverb" (path "/3395a9cf-4e5b-48c0-af92-0653b32bf036" (reference "FS1") (unit 1))))
   )
   (wire (pts (xy 217.17000000000002 119.38) (xy 214.63000000000002 119.38)) (stroke (width 0) (type default)))
@@
     (property "Reference" "LS1" (at 287.02000000000004 179.07 0) (effects (font (size 1.27 1.27)) (justify left)))
     (property "Value" "10in Bulldog" (at 287.02000000000004 181.60999999999999 0) (effects (font (size 1.27 1.27)) (justify left)))
-    (property "Footprint" "Connector_PinHeader_2.54mm:PinHeader_1x02_P2.54mm_Vertical" (at 284.48 186.69 0) (effects (font (size 1.27 1.27)) hide))
+    (property "Footprint" "cambridge_reverb:WirePad_1x02_P5.08mm_D1.5mm" (at 284.48 186.69 0) (effects (font (size 1.27 1.27)) hide))
     (pin "1")
     (pin "2")
-    (instances (project "cambridge_reverb" (path "/bb8f46f8-d0af-4906-93ac-5291092b4687" (reference "LS1") (unit 1))))
+    (instances (project "cambridge_reverb" (path "/3395a9cf-4e5b-48c0-af92-0653b32bf036" (reference "LS1") (unit 1))))
   )
   (wire (pts (xy 279.4 184.15000000000003) (xy 276.86 184.15000000000003)) (stroke (width 0) (type default)))
@@
     (property "Reference" "R_spk_rtn" (at 247.65 179.07 0) (effects (font (size 1.27 1.27)) (justify left)))
     (property "Value" "0R" (at 247.65 181.60999999999999 0) (effects (font (size 1.27 1.27)) (justify left)))
-    (property "Footprint" "Resistor_THT:R_Axial_DIN0207_L6.3mm_D2.5mm_P5.08mm_Vertical" (at 245.11 186.69 0) (effects (font (size 1.27 1.27)) hide))
+    (property "Footprint" "Resistor_THT:R_Axial_DIN0414_L11.9mm_D4.5mm_P15.24mm_Horizontal" (at 245.11 186.69 0) (effects (font (size 1.27 1.27)) hide))
     (pin "1")
     (pin "2")
-    (instances (project "cambridge_reverb" (path "/bb8f46f8-d0af-4906-93ac-5291092b4687" (reference "R_spk_rtn") (unit 1))))
+    (instances (project "cambridge_reverb" (path "/3395a9cf-4e5b-48c0-af92-0653b32bf036" (reference "R_spk_rtn") (unit 1))))
   )
   (wire (pts (xy 240.03 186.69) (xy 237.49 186.69)) (stroke (width 0) (type default)))
