File: kicad/preamp.kicad_sch (KiCad schematic)
At the start: 18 parts, among them Q1 MMBF5457, Q2 MMBF5457

Commit message: Mixed SMD/THT variant (kicad/smd, 155x90), JFET pin-number fix, THT fully routed
Build profiles: gen_kicad.py / gen_pcb.py / gen_bom.py take --profile tht|smd.
One schematic source; the smd profile remaps footprints and writes a self-
contained KiCad project to kicad/smd/ (cambridge_reverb_smd.*, lib tables one
level up), sized 155 x 90 mm for the Part 7 safe-bet chassis.

SMD (70 parts): 0805 R (1206 for R_reg2), 1206 C <= 100 nF, 1210 for 120 nF /
1 uF / C_zobel, SMA + SOD-123 diodes, SOT-23 JFETs fitted directly.
Deliberately THT: power parts, all electrolytics (standing cans use less board
than SMD cans), DIP-8 sockets for the TL072s, the three bench-trimmed JFET
source resistors, LED, connectors, test points. Parts area 4560 mm^2 -> 48 % of
the 155x90 usable area (THT 60 %).

SMD board specifics: 6 mm margin, 0.6 mm gap, 3 mm channels, pad row clear of
the corner holes; GND pour on both layers (top pour solid to SMD ground pads
only, router sees just the bottom plane so every SMD ground pad gets a via);
HighCurrent/Power classes 2.0/1.0 mm for this board (errata #11 addendum).
Routed: 165/167 connections, 1 DRC error (starved thermal), 109 vias; the two
open items are listed in PCB-NOTES as GUI touches. Eight router settings and
three pour strategies compared; the committed one is the best of them.

Errata #18 (HIGH): the JFET symbol had 2 = Gate / 3 = Source; onsemi's 2N5457
(TO-92) and MMBF5457 (SOT-23) both number the leads 1 D / 2 S / 3 G, so the THT
board would have swapped gate and source on Q1, Q2, Q_rec. Symbol renumbered,
both boards regenerated. THT board re-routed (also fixed the column balance):
166/166 connections, 0 DRC violations, 66 vias -- fully routed.

Also: bom/bom-smd*.csv (spec notes, no invented P/Ns), production/smd/
bom-jlcpcb.csv + position file + README for JLCPCB assembly of the SMD side;
route_board.py --drop-planes and default via cost 60; docs (PCB-NOTES,
PCB-AUDIT, README, CHANGELOG, errata, availability audit, Part 10, kicad and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
Connections:
- net Q1G: now also Q1.3 (G); no longer Q1.2 (G)
- net Q1S: now also Q1.2 (S); no longer Q1.3 (S)
- net Q2G: now also Q2.3 (G); no longer Q2.2 (G)
- net Q2S: now also Q2.2 (S); no longer Q2.3 (S)
Changed lines of the file:
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@@
     (pin "1")
     (pin "2")
-    (instances (project "cambridge_reverb" (path "/1f3009cc-abb9-45b2-8580-e2406931df7f" (reference "C_in_pre") (unit 1))))
+    (instances (project "cambridge_reverb" (path "/e208294b-0fa4-4d29-8122-a9e508076fad" (reference "C_in_pre") (unit 1))))
   )
   (wire (pts (xy 116.84 53.339999999999996) (xy 114.3 53.339999999999996)) (stroke (width 0) (type default)))
@@
     (pin "1")
     (pin "2")
-    (instances (project "cambridge_reverb" (path "/1f3009cc-abb9-45b2-8580-e2406931df7f" (reference "R_g1") (unit 1))))
+    (instances (project "cambridge_reverb" (path "/e208294b-0fa4-4d29-8122-a9e508076fad" (reference "R_g1") (unit 1))))
   )
   (wire (pts (xy 116.84 83.82000000000001) (xy 114.3 83.82000000000001)) (stroke (width 0) (type default)))
@@
     (property "Value" "MMBF5457" (at 175.26 58.419999999999995 0) (effects (font (size 1.27 1.27)) (justify left)))
     (property "Footprint" "Package_TO_SOT_THT:TO-92_Inline" (at 172.72 63.49999999999999 0) (effects (font (size 1.27 1.27)) hide))
-    (pin "2")
-    (pin "1")
     (pin "3")
-    (instances (project "cambridge_reverb" (path "/1f3009cc-abb9-45b2-8580-e2406931df7f" (reference "Q1") (unit 1))))
+    (pin "1")
+    (pin "2")
+    (instances (project "cambridge_reverb" (path "/e208294b-0fa4-4d29-8122-a9e508076fad" (reference "Q1") (unit 1))))
   )
   (wire (pts (xy 165.1 63.49999999999999) (xy 162.56 63.49999999999999)) (stroke (width 0) (type default)))
@@
     (pin "1")
     (pin "2")
-    (instances (project "cambridge_reverb" (path "/1f3009cc-abb9-45b2-8580-e2406931df7f" (reference "R_d1") (unit 1))))
+    (instances (project "cambridge_reverb" (path "/e208294b-0fa4-4d29-8122-a9e508076fad" (reference "R_d1") (unit 1))))
   )
   (wire (pts (xy 167.64 33.019999999999996) (xy 165.1 33.019999999999996)) (stroke (width 0) (type default)))
@@
     (pin "1")
     (pin "2")
-    (instances (project "cambridge_reverb" (path "/1f3009cc-abb9-45b2-8580-e2406931df7f" (reference "R_s1") (unit 1))))
+    (instances (project "cambridge_reverb" (path "/e208294b-0fa4-4d29-8122-a9e508076fad" (reference "R_s1") (unit 1))))
   )
   (wire (pts (xy 167.64 104.14) (xy 165.1 104.14)) (stroke (width 0) (type default)))
@@
     (pin "1")
     (pin "2")
-    (instances (project "cambridge_reverb" (path "/1f3009cc-abb9-45b2-8580-e2406931df7f" (reference "C_s1") (unit 1))))
+    (instances (project "cambridge_reverb" (path "/e208294b-0fa4-4d29-8122-a9e508076fad" (reference "C_s1") (unit 1))))
   )
   (wire (pts (xy 207.01 104.14) (xy 204.46999999999997 104.14)) (stroke (width 0) (type default)))
@@
     (pin "1")
     (pin "2")
-    (instances (project "cambridge_reverb" (path "/1f3009cc-abb9-45b2-8580-e2406931df7f" (reference "C_cpl12") (unit 1))))
+    (instances (project "cambridge_reverb" (path "/e208294b-0fa4-4d29-8122-a9e508076fad" (reference "C_cpl12") (unit 1))))
   )
   (wire (pts (xy 207.01 63.49999999999999) (xy 204.46999999999997 63.49999999999999)) (stroke (width 0) (type default)))
@@
     (pin "1")
     (pin "2")
-    (instances (project "cambridge_reverb" (path "/1f3009cc-abb9-45b2-8580-e2406931df7f" (reference "R_g2") (unit 1))))
+    (instances (project "cambridge_reverb" (path "/e208294b-0fa4-4d29-8122-a9e508076fad" (reference "R_g2") (unit 1))))
   )
   (wire (pts (xy 207.01 88.9) (xy 204.46999999999997 88.9)) (stroke (width 0) (type default)))
@@
     (property "Value" "MMBF5457" (at 260.35 58.419999999999995 0) (effects (font (size 1.27 1.27)) (justify left)))
     (property "Footprint" "Package_TO_SOT_THT:TO-92_Inline" (at 257.81 63.49999999999999 0) (effects (font (size 1.27 1.27)) hide))
-    (pin "2")
-    (pin "1")
     (pin "3")
-    (instances (project "cambridge_reverb" (path "/1f3009cc-abb9-45b2-8580-e2406931df7f" (reference "Q2") (unit 1))))
+    (pin "1")
+    (pin "2")
+    (instances (project "cambridge_reverb" (path "/e208294b-0fa4-4d29-8122-a9e508076fad" (reference "Q2") (unit 1))))
   )
   (wire (pts (xy 250.19 63.49999999999999) (xy 247.64999999999998 63.49999999999999)) (stroke (width 0) (type default)))
@@
     (pin "1")
     (pin "2")
-    (instances (project "cambridge_reverb" (path "/1f3009cc-abb9-45b2-8580-e2406931df7f" (reference "R_d2") (unit 1))))
+    (instances (project "cambridge_reverb" (path "/e208294b-0fa4-4d29-8122-a9e508076fad" (reference "R_d2") (unit 1))))
   )
   (wire (pts (xy 252.72999999999996 33.019999999999996) (xy 250.19 33.019999999999996)) (stroke (width 0) (type default)))
@@
     (pin "1")
     (pin "2")
-    (instances (project "cambridge_reverb" (path "/1f3009cc-abb9-45b2-8580-e2406931df7f" (reference "C_pres") (unit 1))))
+    (instances (project "cambridge_reverb" (path "/e208294b-0fa4-4d29-8122-a9e508076fad" (reference "C_pres") (unit 1))))
   )
   (wire (pts (xy 252.72999999999996 104.14) (xy 250.19 104.14)) (stroke (width 0) (type default)))
@@
     (pin "1")
     (pin "2")
-    (instances (project "cambridge_reverb" (path "/1f3009cc-abb9-45b2-8580-e2406931df7f" (reference "R_s2") (unit 1))))
+    (instances (project "cambridge_reverb" (path "/e208294b-0fa4-4d29-8122-a9e508076fad" (reference "R_s2") (unit 1))))
   )
   (wire (pts (xy 292.09999999999997 88.9) (xy 289.56 88.9)) (stroke (width 0) (type default)))
@@
     (pin "1")
     (pin "2")
-    (instances (project "cambridge_reverb" (path "/1f3009cc-abb9-45b2-8580-e2406931df7f" (reference "C_s2") (unit 1))))
+    (instances (project "cambridge_reverb" (path "/e208294b-0fa4-4d29-8122-a9e508076fad" (reference "C_s2") (unit 1))))
   )
   (wire (pts (xy 292.09999999999997 113.03) (xy 289.56 113.03)) (stroke (width 0) (type default)))
@@
     (pin "1")
     (pin "2")
-    (instances (project "cambridge_reverb" (path "/1f3009cc-abb9-45b2-8580-e2406931df7f" (reference "C_treble") (unit 1))))
+    (instances (project "cambridge_reverb" (path "/e208294b-0fa4-4d29-8122-a9e508076fad" (reference "C_treble") (unit 1))))
   )
   (wire (pts (xy 292.09999999999997 48.26) (xy 289.56 48.26)) (stroke (width 0) (type default)))
@@
     (property "Footprint" "cambridge_reverb:TestPoint_THT_D2.0mm_Label" (at 121.91999999999999 243.84 0) (effects (font (size 1.27 1.27)) hide))
     (pin "1")
-    (instances (project "cambridge_reverb" (path "/1f3009cc-abb9-45b2-8580-e2406931df7f" (reference "TP_Q1D") (unit 1))))
+    (instances (project "cambridge_reverb" (path "/e208294b-0fa4-4d29-8122-a9e508076fad" (reference "TP_Q1D") (unit 1))))
   )
   (wire (pts (xy 121.91999999999999 246.38) (xy 121.91999999999999 248.92)) (stroke (width 0) (type default)))
@@
     (property "Footprint" "cambridge_reverb:TestPoint_THT_D2.0mm_Label" (at 147.32 243.84 0) (effects (font (size 1.27 1.27)) hide))
     (pin "1")
-    (instances (project "cambridge_reverb" (path "/1f3009cc-abb9-45b2-8580-e2406931df7f" (reference "TP_Q2D") (unit 1))))
+    (instances (project "cambridge_reverb" (path "/e208294b-0fa4-4d29-8122-a9e508076fad" (reference "TP_Q2D") (unit 1))))
   )
   (wire (pts (xy 147.32 246.38) (xy 147.32 248.92)) (stroke (width 0) (type default)))
@@
     (property "Footprint" "cambridge_reverb:TestPoint_THT_D2.0mm_Label" (at 172.72 243.84 0) (effects (font (size 1.27 1.27)) hide))
     (pin "1")
-    (instances (project "cambridge_reverb" (path "/1f3009cc-abb9-45b2-8580-e2406931df7f" (reference "TP_PRE_OUT") (unit 1))))
+    (instances (project "cambridge_reverb" (path "/e208294b-0fa4-4d29-8122-a9e508076fad" (reference "TP_PRE_OUT") (unit 1))))
   )
   (wire (pts (xy 172.72 246.38) (xy 172.72 248.92)) (stroke (width 0) (type default)))
@@
     (property "Footprint" "cambridge_reverb:TestPoint_THT_D2.0mm_Label" (at 198.12 243.84 0) (effects (font (size 1.27 1.27)) hide))
     (pin "1")
-    (instances (project "cambridge_reverb" (path "/1f3009cc-abb9-45b2-8580-e2406931df7f" (reference "TP_GND_PRE") (unit 1))))
+    (instances (project "cambridge_reverb" (path "/e208294b-0fa4-4d29-8122-a9e508076fad" (reference "TP_GND_PRE") (unit 1))))
   )
   (wire (pts (xy 198.12 246.38) (xy 198.12 248.92)) (stroke (width 0) (type default)))

Commit message: Tone stack: Bass + Treble (passive James) with a switchable mid cut (errata #20)
The panel has Bass and Treble pots, but the design carried a single treble-cut
"Tone" substitute -- and the recovered preamp coupling was the 470 pF chime cap
alone, a 1.3 kHz high-pass that passed no bass at all. Replace both:

- C_cpl_out 1 uF full-band coupling from Q2's drain; C_treble 470 pF becomes a
  bright cap across the top of the volume pot.
- Passive James (Thomas-Vox) Bass/Treble network -- the originals' topology,
  asymmetric, more cut than boost, kept over an active Baxandall so the amp
  keeps its character -- driven by a TL074 (IC3: input buffer, x2 make-up,
  gyrator, output buffer) on its own mid-rail VBIAS_3. Both pots 250k lin in
  the original holes.
- MID CUT toggle for honky pickups: R_mid + a switched series-resonant gyrator
  shunt (1.86 H simulated + 22 nF): -9.6 dB at ~800 Hz, Q ~0.6, flat when off,
  no DC across the switch. SW_MID sits in the original line-reverse switch
  hole -- no new panel holes.
- SPICE: ac_tonestack.cir rewritten rail-aware (all IC3 nodes 8.50 V, noon
  -0.21 dB, notch -9.65 dB at 796 Hz); sweep_tonestack.cir sweeps both pots
  and the switch; results committed.

Generator / placer / router:
- OPAMP14 and SW_SPST symbols, VB_3 / TMK test points (28), BOM rows for IC3,
  the DIP-14 socket, POT_BASS/POT_TREB, SW_MID.
- gen_pcb: tighter profiles (THT 1.2 mm gap / 3.5 mm channels, SMD 0.4 mm),
  overflow repair by moving width between columns, small parts kept in
  schematic order on the shelves, tone/preamp column weighted wider, TP cells
  6x4.5 with the courtyard flush to the cell, input-jack pads down the LEFT
  edge on the 155x90 board (the bottom edge is ~9 mm short for 13 groups),
  keepout rule areas (2 mm edge frame + M3 hole squares) exported to the
  router.
- route_board: refuse a board without its .kicad_pro (a copy routed away from
  the project came back with 0.2 mm tracks and 400 DRC errors); prune
  zero-length segments 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
Parts:
- removed C_treble: 470pF, Capacitor_THT:C_Disc_D7.5mm_W2.5mm_P5.00mm, symbol cr_primitives:C
- added C_cpl_out: 1uF, Capacitor_THT:C_Disc_D7.5mm_W2.5mm_P5.00mm, symbol cr_primitives:C
Connections:
- net PREAMP_OUT: now also C_cpl_out.2
- net Q2D: now also C_cpl_out.1
Changed lines of the file:
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@@
     (pin "1")
     (pin "2")
-    (instances (project "cambridge_reverb" (path "/04add473-f245-4646-8819-fd87b5bcb2bc" (reference "C_in_pre") (unit 1))))
+    (instances (project "cambridge_reverb" (path "/fc10e795-2655-43ed-88d6-50e214c3afc4" (reference "C_in_pre") (unit 1))))
   )
   (wire (pts (xy 116.84 53.339999999999996) (xy 114.3 53.339999999999996)) (stroke (width 0) (type default)))
@@
     (pin "1")
     (pin "2")
-    (instances (project "cambridge_reverb" (path "/04add473-f245-4646-8819-fd87b5bcb2bc" (reference "R_g1") (unit 1))))
+    (instances (project "cambridge_reverb" (path "/fc10e795-2655-43ed-88d6-50e214c3afc4" (reference "R_g1") (unit 1))))
   )
   (wire (pts (xy 116.84 83.82000000000001) (xy 114.3 83.82000000000001)) (stroke (width 0) (type default)))
@@
     (pin "1")
     (pin "2")
-    (instances (project "cambridge_reverb" (path "/04add473-f245-4646-8819-fd87b5bcb2bc" (reference "Q1") (unit 1))))
+    (instances (project "cambridge_reverb" (path "/fc10e795-2655-43ed-88d6-50e214c3afc4" (reference "Q1") (unit 1))))
   )
   (wire (pts (xy 165.1 63.49999999999999) (xy 162.56 63.49999999999999)) (stroke (width 0) (type default)))
@@
     (pin "1")
     (pin "2")
-    (instances (project "cambridge_reverb" (path "/04add473-f245-4646-8819-fd87b5bcb2bc" (reference "R_d1") (unit 1))))
+    (instances (project "cambridge_reverb" (path "/fc10e795-2655-43ed-88d6-50e214c3afc4" (reference "R_d1") (unit 1))))
   )
   (wire (pts (xy 167.64 33.019999999999996) (xy 165.1 33.019999999999996)) (stroke (width 0) (type default)))
@@
     (pin "1")
     (pin "2")
-    (instances (project "cambridge_reverb" (path "/04add473-f245-4646-8819-fd87b5bcb2bc" (reference "R_s1") (unit 1))))
+    (instances (project "cambridge_reverb" (path "/fc10e795-2655-43ed-88d6-50e214c3afc4" (reference "R_s1") (unit 1))))
   )
   (wire (pts (xy 167.64 104.14) (xy 165.1 104.14)) (stroke (width 0) (type default)))
@@
     (pin "1")
     (pin "2")
-    (instances (project "cambridge_reverb" (path "/04add473-f245-4646-8819-fd87b5bcb2bc" (reference "C_s1") (unit 1))))
+    (instances (project "cambridge_reverb" (path "/fc10e795-2655-43ed-88d6-50e214c3afc4" (reference "C_s1") (unit 1))))
   )
   (wire (pts (xy 207.01 104.14) (xy 204.46999999999997 104.14)) (stroke (width 0) (type default)))
@@
     (pin "1")
     (pin "2")
-    (instances (project "cambridge_reverb" (path "/04add473-f245-4646-8819-fd87b5bcb2bc" (reference "C_cpl12") (unit 1))))
+    (instances (project "cambridge_reverb" (path "/fc10e795-2655-43ed-88d6-50e214c3afc4" (reference "C_cpl12") (unit 1))))
   )
   (wire (pts (xy 207.01 63.49999999999999) (xy 204.46999999999997 63.49999999999999)) (stroke (width 0) (type default)))
@@
     (pin "1")
     (pin "2")
-    (instances (project "cambridge_reverb" (path "/04add473-f245-4646-8819-fd87b5bcb2bc" (reference "R_g2") (unit 1))))
+    (instances (project "cambridge_reverb" (path "/fc10e795-2655-43ed-88d6-50e214c3afc4" (reference "R_g2") (unit 1))))
   )
   (wire (pts (xy 207.01 88.9) (xy 204.46999999999997 88.9)) (stroke (width 0) (type default)))
@@
     (pin "1")
     (pin "2")
-    (instances (project "cambridge_reverb" (path "/04add473-f245-4646-8819-fd87b5bcb2bc" (reference "Q2") (unit 1))))
+    (instances (project "cambridge_reverb" (path "/fc10e795-2655-43ed-88d6-50e214c3afc4" (reference "Q2") (unit 1))))
   )
   (wire (pts (xy 250.19 63.49999999999999) (xy 247.64999999999998 63.49999999999999)) (stroke (width 0) (type default)))
@@
     (pin "1")
     (pin "2")
-    (instances (project "cambridge_reverb" (path "/04add473-f245-4646-8819-fd87b5bcb2bc" (reference "R_d2") (unit 1))))
+    (instances (project "cambridge_reverb" (path "/fc10e795-2655-43ed-88d6-50e214c3afc4" (reference "R_d2") (unit 1))))
   )
   (wire (pts (xy 252.72999999999996 33.019999999999996) (xy 250.19 33.019999999999996)) (stroke (width 0) (type default)))
@@
     (pin "1")
     (pin "2")
-    (instances (project "cambridge_reverb" (path "/04add473-f245-4646-8819-fd87b5bcb2bc" (reference "C_pres") (unit 1))))
+    (instances (project "cambridge_reverb" (path "/fc10e795-2655-43ed-88d6-50e214c3afc4" (reference "C_pres") (unit 1))))
   )
   (wire (pts (xy 252.72999999999996 104.14) (xy 250.19 104.14)) (stroke (width 0) (type default)))
@@
     (pin "1")
     (pin "2")
-    (instances (project "cambridge_reverb" (path "/04add473-f245-4646-8819-fd87b5bcb2bc" (reference "R_s2") (unit 1))))
+    (instances (project "cambridge_reverb" (path "/fc10e795-2655-43ed-88d6-50e214c3afc4" (reference "R_s2") (unit 1))))
   )
   (wire (pts (xy 292.09999999999997 88.9) (xy 289.56 88.9)) (stroke (width 0) (type default)))
@@
     (pin "1")
     (pin "2")
-    (instances (project "cambridge_reverb" (path "/04add473-f245-4646-8819-fd87b5bcb2bc" (reference "C_s2") (unit 1))))
+    (instances (project "cambridge_reverb" (path "/fc10e795-2655-43ed-88d6-50e214c3afc4" (reference "C_s2") (unit 1))))
   )
   (wire (pts (xy 292.09999999999997 113.03) (xy 289.56 113.03)) (stroke (width 0) (type default)))
@@
   (symbol (lib_id "cr_primitives:C") (at 297.18 48.26 0) (unit 1)
     (in_bom yes) (on_board yes) (dnp no)
-    (property "Reference" "C_treble" (at 299.72 40.64 0) (effects (font (size 1.27 1.27)) (justify left)))
-    (property "Value" "470pF" (at 299.72 43.18 0) (effects (font (size 1.27 1.27)) (justify left)))
+    (property "Reference" "C_cpl_out" (at 299.72 40.64 0) (effects (font (size 1.27 1.27)) (justify left)))
+    (property "Value" "1uF" (at 299.72 43.18 0) (effects (font (size 1.27 1.27)) (justify left)))
     (property "Footprint" "Capacitor_THT:C_Disc_D7.5mm_W2.5mm_P5.00mm" (at 297.18 48.26 0) (effects (font (size 1.27 1.27)) hide))
     (pin "1")
     (pin "2")
-    (instances (project "cambridge_reverb" (path "/04add473-f245-4646-8819-fd87b5bcb2bc" (reference "C_treble") (unit 1))))
+    (instances (project "cambridge_reverb" (path "/fc10e795-2655-43ed-88d6-50e214c3afc4" (reference "C_cpl_out") (unit 1))))
   )
   (wire (pts (xy 292.09999999999997 48.26) (xy 289.56 48.26)) (stroke (width 0) (type default)))
@@
     (property "Footprint" "cambridge_reverb:TestPoint_THT_D2.0mm_Label" (at 121.91999999999999 243.84 0) (effects (font (size 1.27 1.27)) hide))
     (pin "1")
-    (instances (project "cambridge_reverb" (path "/04add473-f245-4646-8819-fd87b5bcb2bc" (reference "TP_Q1D") (unit 1))))
+    (instances (project "cambridge_reverb" (path "/fc10e795-2655-43ed-88d6-50e214c3afc4" (reference "TP_Q1D") (unit 1))))
   )
   (wire (pts (xy 121.91999999999999 246.38) (xy 121.91999999999999 248.92)) (stroke (width 0) (type default)))
@@
     (property "Footprint" "cambridge_reverb:TestPoint_THT_D2.0mm_Label" (at 147.32 243.84 0) (effects (font (size 1.27 1.27)) hide))
     (pin "1")
-    (instances (project "cambridge_reverb" (path "/04add473-f245-4646-8819-fd87b5bcb2bc" (reference "TP_Q2D") (unit 1))))
+    (instances (project "cambridge_reverb" (path "/fc10e795-2655-43ed-88d6-50e214c3afc4" (reference "TP_Q2D") (unit 1))))
   )
   (wire (pts (xy 147.32 246.38) (xy 147.32 248.92)) (stroke (width 0) (type default)))
@@
     (property "Footprint" "cambridge_reverb:TestPoint_THT_D2.0mm_Label" (at 172.72 243.84 0) (effects (font (size 1.27 1.27)) hide))
     (pin "1")
-    (instances (project "cambridge_reverb" (path "/04add473-f245-4646-8819-fd87b5bcb2bc" (reference "TP_PRE_OUT") (unit 1))))
+    (instances (project "cambridge_reverb" (path "/fc10e795-2655-43ed-88d6-50e214c3afc4" (reference "TP_PRE_OUT") (unit 1))))
   )
   (wire (pts (xy 172.72 246.38) (xy 172.72 248.92)) (stroke (width 0) (type default)))
@@
     (property "Footprint" "cambridge_reverb:TestPoint_THT_D2.0mm_Label" (at 198.12 243.84 0) (effects (font (size 1.27 1.27)) hide))
     (pin "1")
-    (instances (project "cambridge_reverb" (path "/04add473-f245-4646-8819-fd87b5bcb2bc" (reference "TP_GND_PRE") (unit 1))))
+    (instances (project "cambridge_reverb" (path "/fc10e795-2655-43ed-88d6-50e214c3afc4" (reference "TP_GND_PRE") (unit 1))))
   )
   (wire (pts (xy 198.12 246.38) (xy 198.12 248.92)) (stroke (width 0) (type default)))
